Commit message: Add files via upload

File: my_ws/my_robot/urdf/drive_controller.xacro (robot description, xacro)
@@ -12,8 +12,6 @@
       <wheelDiameter>0.1</wheelDiameter>
       <!--Limits-->
-      <wheelAcceleration>10</wheelAcceleration>
-      <wheelTorque>100</wheelTorque>
-      <max_wheel_torque>200</max_wheel_torque>
-      <max_wheel_acceleration>10.0</max_wheel_acceleration>
+      <wheelAcceleration>0</wheelAcceleration>
+      <wheelTorque>80</wheelTorque>
       <!--Output-->
       <robotBaseFrame>base_link</robotBaseFrame>

File: my_ws/my_robot/urdf/my_robot.xacro (robot description, xacro)
@@ -27,7 +27,4 @@
     <material>Gazebo/Red</material>
 </gazebo>
-<!--<gazebo reference="camera_link_optical">
-</gazebo>
--->
   <xacro:include filename="$(find my_robot)/urdf/drive_controller.xacro" />
   <xacro:include filename="$(find my_robot)/urdf/robot_core.xacro" />

File: my_ws/my_robot/urdf/robot_core.xacro (robot description, xacro)
@@ -24,5 +24,5 @@
             <origin xyz = "0.15 0 0.075"/>
             <geometry>
-                <box size = "0.3 0.3 0.15"/>
+                <box size = "0.35 0.3 0.15"/>
             </geometry>
         </visual>
@@ -30,5 +30,5 @@
             <origin xyz = "0.15 0 0.075"/>
             <geometry>
-                <box size = "0.3 0.3 0.15"/>
+                <box size = "0.35 0.3 0.15"/>
             </geometry>
         </collision>
@@ -36,5 +36,5 @@
             <mass value="10"/>
             <geometry>
-                <box size = "0.3 0.3 0.15"/>
+                <box size = "0.35 0.3 0.15"/>
             </geometry>
             <origin xyz = "0.15 0 0.075"/>
@@ -50,11 +50,11 @@
         <parent link = "chassis"/>
         <child link = "left_wheel"/>
-        <origin xyz = "0 0.175 0" rpy = "-${pi/2} 0 0 "/>
-        <axis xyz = "0 0 1"/>
+        <origin xyz = "0.09 0.175 0" rpy = "0 0 0 "/>
+        <axis xyz = "0 1 0"/>
     </joint>
     <link name = "left_wheel">
         <visual>
             <material name = "black"/>
-            <origin xyz = "0 0 0"/>
+                <origin xyz = "0 0 0" rpy= "0 ${pi/2} ${pi/2}"/>
             <geometry>
                 <cylinder radius = "0.05" length = "0.04"/>
@@ -62,11 +62,12 @@
         </visual>
          <collision>
-            <geometry>
-                <cylinder radius = "0.05" length = "0.04"/>
-            </geometry>
-        </collision>
-        <inertial>
-            <mass value="1.0"/>
-            <origin xyz="0 0 0" rpy="-${pi/2} 0 0 "/>
+                <origin xyz = "0 0 0" rpy= "0 ${pi/2} ${pi/2}"/>
+            <geometry>
+                <cylinder radius = "0.05" length = "0.04"/>
+            </geometry>
+        </collision>
+        <inertial>
+            <mass value="5.0"/>
+            <origin xyz = "0 0 0" rpy= "0 ${pi/2} ${pi/2}"/>
             <geometry>
 		        <cylinder radius = "0.05" length = "0.04"/>
@@ -83,22 +84,24 @@
         <parent link = "chassis"/>
         <child link = "right_wheel"/>
-        <origin xyz = "0 -0.175 0" rpy = "${pi/2} 0 0 "/>
-        <axis xyz = "0 0 1"/>
+        <origin xyz = "0.09 -0.175 0" rpy = "0 0 0 "/>
+        <axis xyz = "0 1 0"/>
     </joint>
     <link name = "right_wheel">
         <visual>
             <material name = "black"/>
-            <geometry>
-                <cylinder radius = "0.05" length = "0.04"/>
-            </geometry>
-        </visual>
-        <collision>
-            <geometry>
-                <cylinder radius = "0.05" length = "0.04"/>
-            </geometry>
-        </collision>
-        <inertial>
-            <mass value="1.0"/>
-            <origin xyz="0 0 0" rpy="${pi/2} 0 0 "/>
+            <origin xyz = "0 0 0" rpy= "0 ${pi/2} ${pi/2}"/>
+            <geometry>
+                <cylinder radius = "0.05" length = "0.04"/>
+            </geometry>
+        </visual>
+        <collision>
+            <origin xyz = "0 0 0" rpy= "0 ${pi/2} ${pi/2}"/>
+            <geometry>
+                <cylinder radius = "0.05" length = "0.04"/>
+            </geometry>
+        </collision>
+        <inertial>
+            <mass value="5.0"/>
+            <origin xyz = "0 0 0" rpy= "0 ${pi/2} ${pi/2}"/>
             <geometry>
 		        <cylinder radius = "0.05" length = "0.04"/>
@@ -130,5 +133,5 @@
         </collision>
         <inertial>
-            <mass value="1.0"/>
+            <mass value="5.0"/>
             <origin xyz="0 0 0" rpy="0 0 0 "/>
             <geometry>
@@ -161,5 +164,5 @@
         </collision>
         <inertial>
-            <mass value="1"/>
+            <mass value="0.1"/>
             <origin xyz="0 0 0" rpy="0 0 0"/>
             <geometry>
@@ -192,5 +195,5 @@
         </collision>
         <inertial>
-            <mass value="1"/>
+            <mass value="0.1"/>
             <origin xyz="0 0 0" rpy="0 0 0"/>
             <geometry>
